File: SS.sch (EAGLE design)
At the start: 84 parts, among them K1 4052, K2 4052, Q1 SN74AHC-OR, Q2 UMD5N, Q3 UMD5N, Q4 SN74AHC-OR, Q5 BFP460, Q7 NCP553, Q8 TBD, X1 SO-239, X2 SO-239

Commit message: Changed the isolation circuitry
Tip by [u/Nu2Denim/](https://www.reddit.com/user/Nu2Denim/) at [r/rfelectronics](https://www.reddit.com/r/rfelectronics/comments/1h0pffq/help_me_reuse_this_circuit/)
Parts:
- removed C25: 0.01µF, aarf:MURATACAP
- removed C26: 100pF, aarf:MURATACAP
- removed C27: 0.047µF, aarf:MURATACAP
- removed L7: 100µH, aarf:L-0805
- removed Q8: TBD, aarf:BFR193F
- removed R13, R14: 4.7kΩ, rcl:R-US_M1206
- removed R15: 100Ω, rcl:R-US_M1206
- removed R16: 2.2kΩ, rcl:R-US_M1206
- added SW5, SW6: (no value), aarf:PE4259
Connections:
- removed net N$30: C25.2, Q8.B, R13.2, R14.2
- removed net N$33: C27.2, R15.2, R16.1
- net 0: now also SW5.GND, SW5.RF1, SW6.GND, SW6.RF1; no longer C25.1, C27.1, Q8.E, R14.1
- net 13.8V: no longer L7.2
- net 3V: now also SW5.VDD, SW6.VDD
- net N$23: now also SW4.RFC, SW6.RF2; no longer L7.1, R15.1
- net N$29: now also SW1.RFC, SW5.RF2; no longer C26.1, Q8.C, R16.2
- net N$37: now also SW5.RFC; no longer C26.2, SW1.RFC
- net N$40: now also SW6.RFC; no longer SW4.RFC
- net RLY_BYPASS: now also SW5.CTRL, SW6.CTRL; no longer R13.1
Other:
- note added: "ANTENNA-SIDE ISOLATION"
- note added: "RADIO-SIDE ISOLATION"
- note removed: "RX MUTE"
- moved on the sheet: FB6

Commit message: Small minor improvements
* Corrected position of surge arrestor
* Added description for some networks
* Small improvements in component placement
Parts:
- added C25: 390pF, aarf:MURATACAP
- added D4: 0603ESDA2, aarf:0603ESDA2
Connections:
- net N$10 renamed LNA_IN
- net N$12 renamed FULL_BYP
- net N$15 renamed TX_INH
- net N$29 renamed BPF_IN
- net N$38 renamed BPF_OUT
- net N$43 renamed LNA_OUT
- net N$6 renamed LNA_BYPASS
- net UHF_ON renamed BPF_UHF
- removed net GPIO_OVERRIDE: FB6.2, Q4.B
- removed net N$37: K12.S, SW5.RFC
- removed net N$40: K22.S, SW6.RFC
- new net FROM_BPF: D4.C, K22.S, SW6.RFC
- new net LNA_OFF: Q4.Y, SW3.CTRL, SW4.CTRL
- new net N$6: C25.2, SW5.RFC
- new net TO_BPF: C25.1, D1.C, K12.S
- net 0: now also D4.A
- net AMP_OFF: now also FB6.2, Q4.B; no longer Q4.Y, SW3.CTRL, SW4.CTRL
- net N$8: no longer D1.C
Other:
- note added: "LNA CONTROL ON/BYP"
- moved on the sheet: C1, C10, C11, C12, C2, C21, C22, C23, C24, C3, C4, C5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

Commit message: More updates - refinements
* Added RF relays
* Simplified to a single relay driver (more than enough oomph to drive them both)
* New PNP-based driver for TX_GND
* Copious amount of signal direction and comments
Parts:
- removed K1, K2: 4052, relay:4052
- removed Q3: UMD5N, aarf:UMD5N
- removed R8: 10kΩ, rcl:R-US_M1206
- removed SW1: (no value), aarf:PE4259
- added RL1: ANT_RLY, aarf:RELAY-TE-HF3
- added RL2: RADIO_RLY, aarf:RELAY-TE-HF3
- added SW_SEL_V/U-IN: PE4259, aarf:PE4259
- added T1: MMBTRA104SS, transistor:MUN2111T1-PNP_DRIVER-SC59-BEC
- PAD3: value RX -> TX_GND
- Q6: value (none) -> L78L05
- SW_ISOL-ANT, SW_ISOL-RADIO, SW_SEL_LNA-IN, SW_SEL_LNA-OUT, SW_SEL_V/U-OUT: value (none) -> PE4259
- renumbered SW2 to SW_SEL_V/U-OUT, SW3 to SW_SEL_LNA-IN, SW4 to SW_SEL_LNA-OUT, SW5 to SW_ISOL-ANT, SW6 to SW_ISOL-RADIO
Connections:
- net N$23 renamed LNA-SW_OUT
- removed net 1: C18.1, D3.A, K21.2, R10.2
- removed net BPF_UHF: FB5.2, SW1.CTRL, SW_SEL_V/U-OUT.CTRL
- removed net FROM_BPF: D4.C, K22.S, SW_ISOL-RADIO.RFC
- removed net FULL_BYP: K12.O, K22.O
- removed net N$11: Q2.4, R9.1
- removed net N$2: K22.P, X2.1
- removed net N$34: C17.2, D2.C, K11.2, R9.2
- removed net N$35: Q3.2, Q3.3
- removed net N$39: Q3.4, R10.1
- removed net N$8: K12.P, X1.1
- removed net TX_INH: FB2.2, K13.P, K23.O
- removed net TX_OFF: FB3.2, Q1.A
- new net AMP+BPF_OUT: D4.C, RL2.14, SW_ISOL-RADIO.RFC
- new net ANTENNA: RL1.6, X1.1
- new net DRIVE_TX: FB3.2, T1.B
- new net N$30: R10.2, RL2.1
- new net RADIO: RL2.6, X2.1
- new net RADIO_TX: Q1.A, T1.C
- new net RELAY-TO-RELAY_BYPASS: RL1.20, RL2.20
- new net RELAY_PWR: C17.2, C18.1, D2.C, D3.C, FB2.2, Q2.4, R10.1, R9.1
- new net SEL_BPF_UHF: FB5.2, SW_SEL_V/U-IN.CTRL, SW_SEL_V/U-OUT.CTRL
- net 0: now also D3.A, RL1.10, RL1.11, RL1.12, RL1.13, RL1.15, RL1.17, RL1.19, RL1.2, RL1.21, RL1.22, RL1.5, RL1.7, RL2.10, RL2.11, RL2.12, RL2.13, RL2.15, RL2.17, RL2.19, RL2.2, RL2.21, RL2.22, RL2.5, RL2.7, SW_SEL_V/U-IN.GND; no longer D3.C, K11.1, K13.O, K21.1, K23.P, Q3.6, SW1.GND
- net 13.8V: no longer Q3.1, R8.1
- net 3V: now also SW_SEL_V/U-IN.VDD, T1.E; no longer SW1.VDD
- net BPF_IN: now also SW_SEL_V/U-IN.RFC; no longer SW1.RFC
- net N$1: now also R9.2, RL1.1; no longer K13.S, R8.2
- net N$3: now also SW_SEL_V/U-IN.RF1; no longer SW1.RF1
- net N$4: now also SW_SEL_V/U-IN.RF2; no longer SW1.RF2
- net RLY_BYPASS: no longer Q3.5
- net TO_BPF: now also RL1.14; no longer K12.S
Other:
- note added: "ANT-SIDE RELAY"
- note removed: "ANTENNA-SIDE RELAY"
- moved on the sheet: C17, C18, D1, D2, D3, D4, Q1, Q2, R10, R9, X1, X2

Commit message: Progress.
Schematic:
* Added pulldown resistors to input ports at OR comparator
* Added static bleeding on antenna-side isolation
* Replaced some 1206 caps with 0805

Board:
* Started arranging the first components.
Parts:
- removed X1, X2: SO-239, aarf:SO-239
- added ANTENNA: ANTENNA, wirepad:SMD2
- added L7: 1000µH, aarf:L-0805
- added R13, R14: 10kΩ, rcl:R-US_M1206
- added R8: 1kΩ, rcl:R-US_M1206
- added RADIO: RADIO, wirepad:SMD2
- 13.8V, TX_INH: SPICEPREFIX (none) -> X
- C1, C2: device rcl:C-EUC0805 -> aarf:MURATACAP
- D2, D3: value (none) -> 1N4148
- F1: value (none) -> 1231; SPICEPREFIX (none) -> B
- FB1, FB2, FB3, FB4, FB5, FB6: value (none) -> BLM21
- renumbered PAD1 to 13.8V, PAD2 to TX_INH, PAD3 to TX_GND, PAD4 to GND, PAD5 to BYPASS, PAD6 to UHF, PAD7 to AMP_OFF
Connections:
- new net N$2: L7.1, R8.1
- net 0: no longer C1.1, C10.2, C11.2, C14.1, C15.1, C16.1, C17.1, C18.2, C19.1, C2.1, C20.1, C21.1, C22.1, C23.1, C24.1, C3.1, C6.1, C7.1, D1.A, D2.A, D3.A, D4.A, L2.2, L4.2, Q1.GND, Q2.6, Q4.GND, Q5.E, Q6.GND, Q7.GN, RL1.10, RL1.11, RL1.12, RL1.13, RL1.15, RL1.17, RL1.19, RL1.2, RL1.21, RL1.22, RL1.5, RL1.7, RL2.10, RL2.11, RL2.12, RL2.13, RL2.15, RL2.17, RL2.19, RL2.2, RL2.21, RL2.22, RL2.5, RL2.7, SW_ISOL-ANT.GND, SW_ISOL-ANT.RF1, SW_ISOL-RADIO.GND, SW_ISOL-RADIO.RF1, SW_SEL_LNA-IN.GND, SW_SEL_LNA-OUT.GND, SW_SEL_V/U-IN.GND, SW_SEL_V/U-OUT.GND, X1.2, X2.2
- net ANTENNA: now also ANTENNA.P; no longer X1.1
- net EXT_BYPASS: now also R14.1
- net GND: now also C1.1, C10.2, C11.2, C14.1, C15.1, C16.1, C17.1, C18.2, C19.1, C2.1, C20.1, C21.1, C22.1, C23.1, C24.1, C3.1, C6.1, C7.1, D1.A, D2.A, D3.A, D4.A, L2.2, L4.2, L7.2, Q1.GND, Q2.6, Q4.GND, Q5.E, Q6.GND, Q7.GN, R13.2, R14.2, RL1.10, RL1.11, RL1.12, RL1.13, RL1.15, RL1.17, RL1.19, RL1.2, RL1.21, RL1.22, RL1.5, RL1.7, RL2.10, RL2.11, RL2.12, RL2.13, RL2.15, RL2.17, RL2.19, RL2.2, RL2.21, RL2.22, RL2.5, RL2.7, SW_ISOL-ANT.GND, SW_ISOL-ANT.RF1, SW_ISOL-RADIO.GND, SW_ISOL-RADIO.RF1, SW_SEL_LNA-IN.GND, SW_SEL_LNA-OUT.GND, SW_SEL_V/U-IN.GND, SW_SEL_V/U-OUT.GND
- net RADIO: now also RADIO.P; no longer X2.1
- net RADIO_TX: now also R13.1
- net TO_BPF: now also R8.2
Other:
- moved on the sheet: C17, D1, D2, D4, R9, RL1, SW_ISOL-RADIO
