File: CAD/SS.sch (EAGLE design)
At the start: 133 parts, among them Q1 SN74AHC-NOR, Q2 UMD5N, Q3 MIC5205, Q4 SN74AHC-AND, Q5 BFP460, Q6 TCR1HF50, T1 MMBTRA104SS, X1 ANTENNA, X2 RADIO, X3 INP, X4 AMP-O, X5 BPF-O

Commit message: Releasing: Revision F
* Improved UHF BPF.
* Changed "Bypass" and "VHF/UHF" input selectors from 3V to 5V via
  resisitive divisors.
* Added u.FL calibration pads.
* Updated documentation, BOM, images, tests
* Resolves #30
Parts:
- removed C34: 2.4pF, aarf:C-0805
- added R11, R16: 100Ω, aarf:R-1206
- added R18: 10kΩ, aarf:R-1206
- added X10: CAL-T1, adafruit:ANTENNA_U.FL
- added X6: CAL-O, adafruit:ANTENNA_U.FL
- added X7: CAL-S, adafruit:ANTENNA_U.FL
- added X8: CAL-L, adafruit:ANTENNA_U.FL
- added X9: CAL-T2, adafruit:ANTENNA_U.FL
- C3: value 18pF -> 19.5pF
- C33, C35: value 4.7pF -> 8.2pF
- C47: value 8.2pF -> 2.4pF
- C6, C7: value 20pF -> 18pF
- R14, R17: value 10kΩ -> 15kΩ
- R7: value 1kΩ -> 10kΩ
Connections:
- removed net 1.86PF: C34.2, C47.1
- new net N$10: R11.2, R16.2, X8.GND@0, X8.GND@1
- new net N$12: FB5.1, R18.1
- new net N$14: X10.SIGNAL, X9.SIGNAL
- new net N$8: X7.GND@0, X7.GND@1, X7.SIGNAL
- new net N$9: R11.1, R16.1, X8.SIGNAL
- net GND: now also X10.GND@0, X10.GND@1, X9.GND@0, X9.GND@1
- net UHF-P1: now also C47.1; no longer C34.1
- net VHF_ON_IN: now also R18.2; no longer FB5.1
Other:
- note added: "ANTENNA-SIDE PROTECTION"
- note added: "U.FL CALIBRATION STANDARDS"
- note removed: "ANTENNA-SIDE ISOLATION"
- moved on the sheet: C47, R14
